File: pcb/Denshi_fuka.kicad_sch (KiCad schematic)
At the start: 21 parts, among them J1 Power, J2 Digital/PWM, J3 Analog, J4 Digital/PWM, Q1 NMOS, Q2 NMOS, U1 LM358, U3 ADS1115IDGS, U4 MCP6002-xP, U5 MCP4728, U6 ISO1540

Commit message: schematic completed!
Parts:
- removed U3: ADS1115IDGS, Package_SO:TSSOP-10_3x3mm_P0.5mm, symbol Analog_ADC:ADS1115IDGS
- removed U5: MCP4728, Package_SO:MSOP-10_3x3mm_P0.5mm, symbol Analog_DAC:MCP4728
- removed U6: ISO1540, Package_SO:SOIC-8_3.9x4.9mm_P1.27mm, symbol Isolator:ISO1540
- added C1, C2, C4, C6: 0.1uF, Capacitor_THT:C_Disc_D5.0mm_W2.5mm_P5.00mm, symbol Device:C
- added C3, C7, C8: C, symbol Device:C
- added C5: 1uF, Capacitor_THT:C_Disc_D5.0mm_W2.5mm_P5.00mm, symbol Device:C
- added F3, F4: Fuse, symbol Device:Fuse
- added J10, J11: Conn_01x02_Socket, symbol Connector:Conn_01x02_Socket
- added J5: SCREW TERMINAL, symbol Connector:Conn_01x02_Socket
- added J6, J7, J8, J9: SCREW TERMINAL, symbol Connector:Conn_01x01_Socket
- added R1: 1MΩ, Resistor_THT:R_Axial_DIN0207_L6.3mm_D2.5mm_P10.16mm_Horizontal, symbol Device:R
- added R2: 240kΩ, Resistor_THT:R_Axial_DIN0207_L6.3mm_D2.5mm_P10.16mm_Horizontal, symbol Device:R
- added R3: 1.5MΩ, Resistor_THT:R_Axial_DIN0207_L6.3mm_D2.5mm_P10.16mm_Horizontal, symbol Device:R
- added R4: 24kΩ, Resistor_THT:R_Axial_DIN0207_L6.3mm_D2.5mm_P10.16mm_Horizontal, symbol Device:R
- added R5, R6: 10kΩ, symbol Device:R
- added U2: MCP4822, Package_DIP:DIP-8_W7.62mm_Socket_LongPads, symbol Analog_DAC:MCP4822
- added U3: MCP3564R, symbol Fuka_sym:MCP3564R
- added U5: Si8651, symbol Fuka_sym:Si8651
- added U7: LEG_3V3, Package_TO_SOT_THT:TO-220-3_Vertical, symbol Regulator_Linear:LM7805_TO220
- Cf1: renamed from Cf; footprint (none) -> Capacitor_THT:C_Disc_D5.0mm_W2.5mm_P5.00mm
- Cf2: renamed from Cf1; footprint (none) -> Capacitor_THT:C_Disc_D5.0mm_W2.5mm_P5.00mm
- D1, D2: footprint (none) -> Package_TO_SOT_THT:TO-220-2_Vertical
- Q1, Q2: value NMOS -> 2SK3176; footprint (none) -> Package_TO_SOT_THT:TO-247-3_Horizontal_TabUp
- Rf1: renamed from Rf; footprint (none) -> Resistor_THT:R_Axial_DIN0207_L6.3mm_D2.5mm_P10.16mm_Horizontal
- Rf2: renamed from Rf1; footprint (none) -> Resistor_THT:R_Axial_DIN0207_L6.3mm_D2.5mm_P10.16mm_Horizontal
- Rg1: renamed from Rg; footprint (none) -> Resistor_THT:R_Axial_DIN0207_L6.3mm_D2.5mm_P10.16mm_Horizontal
- Rg2: renamed from Rg1; footprint (none) -> Resistor_THT:R_Axial_DIN0207_L6.3mm_D2.5mm_P10.16mm_Horizontal
- Rsense1: renamed from Rsense; footprint (none) -> Resistor_THT:R_Axial_Power_L48.0mm_W12.5mm_P55.88mm
- Rsense2: renamed from Rsense1; footprint (none) -> Resistor_THT:R_Axial_Power_L48.0mm_W12.5mm_P55.88mm
- U4: footprint (none) -> Package_DIP:DIP-8_W7.62mm_Socket_LongPads
Connections:
- net +3V3: now also R5.1, R6.1; no longer J1.4 (Pin_4)
- net +5V: now also C1.1, U5.1 (VDD1), U5.7 (EN1)
- net MISO/PB4: now also U5.6 (A5)
- net MOSI/PB3: now also U5.3 (A2)
- net PB1: now also U5.5 (A4)
- net PB2: now also U5.4 (A3)
- net SCK/PB5: now also U5.2 (A1)
- net VDC1: now also D1.1 (K), Q1.1 (D), F3.1; no longer D1.2 (A)
- net VDC2: now also D2.1 (K), Q2.1 (D), F4.1, R3.1; no longer D2.2 (A)
- net ADC_i2+: now reaches Q2.3 (S), Rf2.2, Rsense2.1
- net ADC_i2+: now also U3.7 (CH2)
- net ADC_i1+: now reaches Q1.3 (S), Rf1.2, Rsense1.1
- net ADC_i1+: now also U3.5 (CH0)
- net at U4.5 (+): now also R3.2, R4.1
- net GNDA: now reaches U4.6 (-)
- net GNDA: now also D1.2 (A), D2.2 (A), Rsense1.2, Rsense2.2, U1.4 (V-), U4.2 (-), U4.4 (V-), C2.2, C3.2, C4.2, C5.2, C6.2, C7.2, C8.2, J10.2 (Pin_2), J11.2 (Pin_2), J5.2 (Pin_2), J9.1 (Pin_1), R2.2, R4.2, U2.5 (~{LDAC}), U2.7 (Vss), U3.18 (MCLK), U3.19 (DGND), U3.2 (AGND), U3.3 (REFIN-), U3.6 (CH1), U3.8 (CH3), U5.9 (GND2), U7.2 (GND)
- net ADC_v2: now reaches U4.7
- net ADC_v2: now also U3.10 (CH5)
- net Vout1: now reaches U1.3 (+)
- net Vout1: now also U2.8 (VA)
- net Vout2: now reaches U1.5 (+)
- net Vout2: now also U2.6 (VB)
- net ADC_v1: now reaches U4.1
- net ADC_v1: now also U3.9 (CH4)
- net at U4.3 (+): now also R1.2, R2.1
- removed net GND: J1.6 (Pin_6), J1.7 (Pin_7), J2.4 (Pin_4), Rsense1.2, Rsense2.2, U1.4 (V-), U4.4 (V-)
- removed net VCC: J1.8 (Pin_8), U1.8 (V+), U4.8 (V+)
- new net: F4.2, J7.1 (Pin_1)
- new net: F3.2, J6.1 (Pin_1)
- new net: C4.1, U3.4 (REFIN+/OUT)
- new net +12V: C7.1, J5.1 (Pin_1), U1.8 (V+), U7.1 (VI)
- new net +3V3_A: C2.1, C3.1, C5.1, C6.1, C8.1, U2.1 (Vdd), U3.1 (AVDD), U3.20 (DVDD), U4.8 (V+), U5.10 (EN2), U5.16 (VDD2), U7.3 (VO)
- new net CS_MCP3564: U3.13 (~{CS}), U5.13 (B3)
- new net CS_MCP4822: U2.2 (~{CS}), U5.12 (B4)
- new net GNDD: C1.2, J1.6 (Pin_6), J1.7 (Pin_7), J2.4 (Pin_4), U5.8 (GND1)
- new net SCK: U2.3 (SCK), U3.14 (SCK), U5.15 (B1)
- new net SDI: U2.4 (SDI), U3.15 (SDI), U5.14 (B2)
- new net SDO: U3.16 (SDO), U5.11 (B5)
- new net Thermo_1: J10.1 (Pin_1), R6.2, U3.11 (CH6)
- new net Thermo_2: J11.1 (Pin_1), R5.2, U3.12 (CH7)
- new net VDC1_Sense: R1.1
- new net VDC1_sense: J8.1 (Pin_1)
- new net Vin: J1.8 (Pin_8)
- no-connect marks 1 -> 4
Other:
- note added: "Electrically Isolated"
- moved on the sheet: Cf1, Cf2, Q1, Q2, Rf1, Rf2, Rg1, Rg2, Rsense1, Rsense2, U1A, U1B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

Commit message: modify sch
Parts:
- added D1, D4: D_Zener, symbol Device:D_Zener
- added R2, R5: 1kΩ, symbol Device:R
- added Rpd1, Rpd2: 100kΩ, symbol Device:R
- renumbered C7 to C3, C8 to C4, C4 to C7, C3 to C8, D1 to D2, D2 to D3, F3 to F1, F4 to F2, J6 to J1, J11 to J10, J5 to J11, J8 to J2, J2 to J3, J7 to J4, J1 to J5, J9 to J6, J10 to J7, J3 to J8, J4 to J9, R2 to R3, R3 to R4, R4 to R6, R6 to R7, R5 to R8, U7 to U1, U1 to U2, U4 to U3, U5 to U4, U3 to U5, U2 to U6
Connections:
- net ADC_i1+: now also D1.1 (K), R2.2; no longer Q1.3 (S), Rf1.2, Rsense1.1
- net ADC_i2+: now also D4.1 (K), R5.2; no longer Q2.3 (S), Rf2.2, Rsense2.1
- net GNDA: now also D1.2 (A), D4.2 (A), Rpd1.2, Rpd2.2
- net at Q1.2 (G), Rg1.2: now also Rpd1.1
- net at Q2.2 (G), Rg2.2: now also Rpd2.1
- new net: Q1.3 (S), R2.1, Rf1.2, Rsense1.1
- new net: Q2.3 (S), R5.1, Rf2.2, Rsense2.1
Other:
- note added: "3.3V Regurator"
- note added: "ADC"
- note added: "Analog Power Input"
- note added: "Connect to Arduino"
- note added: "DAC"
- note added: "Digital Isolator"
- note added: "Interface Connector"
- note added: "Main Current Controll Circuit"
- note added: "Reverse Voltage Bypass Diode"
- note added: "Thermistor Connector"
- moved on the sheet: Cf1, Cf2, D2, D3, F1, F2, J1, J10, J11, J2, J4, J6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

Commit message: add some circuit
Parts:
- added D5: D, symbol Device:D
- added J12: FAN_CONN1, symbol Connector:Conn_01x04_Socket
- added J13: FAN_CONN2, symbol Connector:Conn_01x04_Socket
- added K1: Relay, symbol Relay:Relay_SPST-NO
- added Q3: NPN, symbol Simulation_SPICE:NPN
- added R10, R9: 470Ω, symbol Device:R
- added R11, R12: 10kΩ, symbol Device:R
- added R13, R14, Rb: 1kΩ, symbol Device:R
- added U10, U7, U8, U9: PC817, symbol Isolator:Optocoupler_DC_PhotoNPN_AKEC
- U3: value MCP6002-xP -> MCP6002
Connections:
- net +12V: now also J12.2 (Pin_2), J13.2 (Pin_2), K1.13, R13.2, R14.1; no longer J11.1 (Pin_1)
- net +5V: now also D5.1 (K), K1.A1, R11.2, R12.2
- net GNDA: now also J12.1 (Pin_1), J13.1 (Pin_1), U7.3, U8.3
- net GNDD: now also Q3.3 (E), U10.3, U7.2, U8.2, U9.3
- net PB0: now also Rb.2
- net PD2: now also R11.1, U10.4
- net PD3: now also R12.1, U9.4
- net PD5: now also R9.1
- net PD6: now also R10.1
- new net: R9.2, U7.1
- new net: R13.1, U9.1
- new net: D5.2 (A), K1.A2, Q3.1 (C)
- new net: Q3.2 (B), Rb.1
- new net: R10.2, U8.1
- new net: R14.2, U10.1
- new net +12V_in: J11.1 (Pin_1), K1.14
- new net FAN_PWM1: J12.4 (Pin_4), U7.4
- new net FAN_PWM2: J13.4 (Pin_4), U8.4
- new net FAN_TACH1: J12.3 (Pin_3), U10.2
- new net FAN_TACH2: J13.3 (Pin_3), U9.2
Other:
- note added: "Power Control Relay"
- moved on the sheet: C1, C2, C3, C4, C5, C6, C7, C8, Cf1, Cf2, D1, D2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

Commit message: Fuck
Parts:
- removed C3, C4: C, symbol Device:C
- removed J5: Power, Connector_PinSocket_2.54mm:PinSocket_1x08_P2.54mm_Vertical, symbol Connector_Generic:Conn_01x08
- removed J8: Analog, Connector_PinSocket_2.54mm:PinSocket_1x06_P2.54mm_Vertical, symbol Connector_Generic:Conn_01x06
- removed J9: Digital/PWM, Connector_PinSocket_2.54mm:PinSocket_1x08_P2.54mm_Vertical, symbol Connector_Generic:Conn_01x08
- removed K1: Relay, symbol Relay:Relay_SPST-NO
- added C3, C4: 10uF, Capacitor_THT:CP_Radial_D5.0mm_P2.00mm, symbol Device:C_Polarized
- added J1, J4: Conn_01x08, Connector_PinHeader_2.54mm:PinHeader_1x08_P2.54mm_Vertical, symbol Connector_Generic:Conn_01x08
- added J2: Conn_01x06, Connector_PinHeader_2.54mm:PinHeader_1x06_P2.54mm_Vertical, symbol Connector_Generic:Conn_01x06
- added K2: SRD05VDCSLC, Relay_THT:Relay_SPDT_SANYOU_SRD_Series_Form_C, symbol Relay:SANYOU_SRD_Form_C
- added Rjp1, Rjp2: 0Ω, Resistor_THT:R_Axial_DIN0309_L9.0mm_D3.2mm_P12.70mm_Horizontal, symbol Device:R
- C5: renamed from C8; value C -> 0.1uF; footprint (none) -> Capacitor_THT:C_Disc_D5.0mm_W2.5mm_P5.00mm
- C6: renamed from C5; footprint Capacitor_THT:C_Disc_D5.0mm_W2.5mm_P5.00mm -> Capacitor_THT:C_Disc_D3.0mm_W1.6mm_P2.50mm
- D3: renamed from D5; value D -> 1N4148; footprint (none) -> Diode_THT:D_DO-35_SOD27_P7.62mm_Horizontal
- D4: renamed from D1; value D_Zener -> D_Zener_3V3; footprint (none) -> Diode_THT:D_DO-35_SOD27_P7.62mm_Horizontal
- D5: renamed from D4; value D_Zener -> D_Zener_3V3; footprint (none) -> Diode_THT:D_DO-35_SOD27_P7.62mm_Horizontal
- F1, F2: footprint (none) -> MyParts:MF-563
- J10: renamed from J7; value Conn_01x02_Socket -> JST_PH2P; footprint (none) -> Connector_JST:JST_PH_B2B-PH-K_1x02_P2.00mm_Vertical
- J11: renamed from J10; value Conn_01x02_Socket -> JST_PH2P; footprint (none) -> Connector_JST:JST_PH_B2B-PH-K_1x02_P2.00mm_Vertical
- J12, J13: footprint (none) -> Connector:FanPinHeader_1x04_P2.54mm_Vertical
- J3: value Digital/PWM -> Conn_01x10; footprint Connector_PinSocket_2.54mm:PinSocket_1x10_P2.54mm_Vertical -> Connector_PinHeader_2.54mm:PinHeader_1x10_P2.54mm_Vertical
- J5: renamed from J11; footprint (none) -> TerminalBlock_Phoenix:TerminalBlock_Phoenix_PT-1,5-2-5.0-H_1x02_P5.00mm_Horizontal
- J6: renamed from J1; footprint (none) -> Aki-Parts:PCB-20
- J7: renamed from J2; footprint (none) -> Aki-Parts:PCB-20
- J8: renamed from J4; footprint (none) -> Aki-Parts:PCB-20
- J9: renamed from J6; footprint (none) -> Aki-Parts:PCB-20
- Q1: renamed from Q3; value NPN -> 2SC1815; footprint (none) -> Package_TO_SOT_THT:TO-92_Inline
- R1: renamed from R12; footprint (none) -> Resistor_THT:R_Axial_DIN0207_L6.3mm_D2.5mm_P10.16mm_Horizontal
- R10: renamed from R5; footprint (none) -> Resistor_THT:R_Axial_DIN0207_L6.3mm_D2.5mm_P10.16mm_Horizontal
- R11: renamed from R4; value 1.5MΩ -> 1MΩ
- R12: renamed from R6; value 24kΩ -> 10kΩ
- R13: renamed from R1; value 1MΩ -> 100kΩ
- R14: renamed from R3; value 240kΩ -> 22kΩ
- R2: renamed from R11; footprint (none) -> Resistor_THT:R_Axial_DIN0207_L6.3mm_D2.5mm_P10.16mm_Horizontal
- R3: renamed from R13; footprint (none) -> Resistor_THT:R_Axial_DIN0207_L6.3mm_D2.5mm_P10.16mm_Horizontal
- R4: renamed from R14; footprint (none) -> Resistor_THT:R_Axial_DIN0207_L6.3mm_D2.5mm_P10.16mm_Horizontal
- R5: renamed from R10; value 470Ω -> 220Ω; footprint (none) -> Resistor_THT:R_Axial_DIN0207_L6.3mm_D2.5mm_P10.16mm_Horizontal
- R6: renamed from R9; value 470Ω -> 220Ω; footprint (none) -> Resistor_THT:R_Axial_DIN0207_L6.3mm_D2.5mm_P10.16mm_Horizontal
- R7, R8, Rpd1, Rpd2: footprint (none) -> Resistor_THT:R_Axial_DIN0207_L6.3mm_D2.5mm_P10.16mm_Horizontal
- R9: renamed from R2; footprint (none) -> Resistor_THT:R_Axial_DIN0207_L6.3mm_D2.5mm_P10.16mm_Horizontal
- Rb1: renamed from Rb; footprint (none) -> Resistor_THT:R_Axial_DIN0207_L6.3mm_D2.5mm_P10.16mm_Horizontal
- Rf1, Rf2, Rg1, Rg2: footprint Resistor_THT:R_Axial_DIN0207_L6.3mm_D2.5mm_P10.16mm_Horizontal -> Resistor_THT:R_Axial_DIN0309_L9.0mm_D3.2mm_P12.70mm_Horizontal
- Rsense1: value 0.1Ω 5W -> 0.1Ω 10W
- Rsense2: value 10Ω 5W -> 10Ω 10W
- U1: renamed from U4; footprint (none) -> MyParts:DIP-16_W15.24mm (600mil)
- U10: renamed from U5; footprint (none) -> MyParts:DIP-20_W15.24mm_Socket_LongPads
- U2: renamed from U1; value LEG_3V3 -> LM2940T-3.3
- U4: renamed from U3; value MCP6002 -> MCP6232
- U5: renamed from U9; value PC817 -> PS817; footprint (none) -> Package_DIP:DIP-4_W7.62mm_LongPads
- U6: renamed from U10; value PC817 -> PS817; footprint (none) -> Package_DIP:DIP-4_W7.62mm_LongPads
- U7: renamed from U8; value PC817 -> PS817; footprint (none) -> Package_DIP:DIP-4_W7.62mm_LongPads
- U8: renamed from U7; value PC817 -> PS817; footprint (none) -> Package_DIP:DIP-4_W7.62mm_LongPads
- renumbered C6 to C7, C7 to C8, D2 to D1, D3 to D2, Q1 to Q2, Q2 to Q3, U2 to U3, U6 to U9
Connections:
- net +3V3 is gone; now on net +3V3_A: R7.1, R8.1
- net VDC1_sense is gone; now on net VDC1_Sense: J7.1 (Pin_1)
- net +12V: now also R3.1, C3.1, K2.1; no longer R3.2
- net +12V_in: now also K2.3
- net +3V3_A: now also C4.1
- net +5V: now also J1.5 (Pin_5), K2.5
- net ADC_i1+: now also U10.7 (CH2); no longer U10.5 (CH0)
- net ADC_i2+: now also U10.5 (CH0); no longer U10.7 (CH2)
- net CS_MCP3564: now also Rjp2.1; no longer U10.13 (~{CS})
- net CS_MCP4822: now also Rjp1.1; no longer U9.2 (~{CS})
- net GNDA: now also C3.2, C4.2
- net GNDD: now also J1.6 (Pin_6), J1.7 (Pin_7)
- net IOREF: now also J1.2 (Pin_2)
- net PB0: no longer Rb1.2
- net PC0: now also Rb1.1, J2.1 (Pin_1)
- net PC1: now also J2.2 (Pin_2)
- net PC2: now also J2.3 (Pin_3)
- net PC3: now also J2.4 (Pin_4)
- net PD2: now also J4.6 (Pin_6)
- net PD3: now also J4.5 (Pin_5)
- net PD4: now also J4.4 (Pin_4)
- net PD5: now also J4.3 (Pin_3)
- net PD6: now also J4.2 (Pin_2)
- net PD7: now also J4.1 (Pin_1)
- net RXD/PD0: now also J4.8 (Pin_8)
- net SCL/PC5: now also J2.6 (Pin_6)
- net SDA/PC4: now also J2.5 (Pin_5)
- net TXD/PD1: now also J4.7 (Pin_7)
- net VDC1: now also Q2.2 (D); no longer Q2.1 (D)
- net VDC2: now also Q3.2 (D); no longer Q3.1 (D)
- net Vin: now also J1.8 (Pin_8)
- net ~{RESET}: now also J1.3 (Pin_3)
- net at U5.1: now also R3.2; no longer R3.1
- net at D3.2 (A), Q1.1 (C): now also K2.2
- net at Rg2.2, Rpd2.1: now also Q3.1 (G); no longer Q3.2 (G)
- net at Q1.2 (B): now also Rb1.2; no longer Rb1.1
- net at Rg1.2, Rpd1.1: now also Q2.1 (G); no longer Q2.2 (G)
- new net: Rjp1.2, U9.2 (~{CS})
- new net: Rjp2.2, U10.13 (~{CS})
- no-connect marks 4 -> 5
Other:
- note added: "Fan Connector"
- note added: "Fan Signal Isolator"
- note added: "Specification"
- note added: "Voltage Follower Amp"
- moved on the sheet: C1, C2, C5, C6, C7, C8, Cf1, Cf2, D1, D2, D3, D4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

Commit message: pcb kansei
Parts:
- removed Rjp1: 0Ω, Resistor_THT:R_Axial_DIN0309_L9.0mm_D3.2mm_P12.70mm_Horizontal, symbol Device:R
- added Rjp3, Rjp4: 0Ω, Resistor_THT:R_Axial_DIN0207_L6.3mm_D2.5mm_P15.24mm_Horizontal, symbol Device:R
- Rjp2: footprint Resistor_THT:R_Axial_DIN0309_L9.0mm_D3.2mm_P12.70mm_Horizontal -> Resistor_THT:R_Axial_DIN0309_L9.0mm_D3.2mm_P15.24mm_Horizontal
- Rpd1, Rpd2: footprint Resistor_THT:R_Axial_DIN0207_L6.3mm_D2.5mm_P10.16mm_Horizontal -> Resistor_THT:R_Axial_DIN0207_L6.3mm_D2.5mm_P15.24mm_Horizontal
Connections:
- net CS_MCP4822: now also U9.2 (~{CS})
- net GNDA: now also Rjp3.2, Rjp4.2; no longer U10.6 (CH1), U10.8 (CH3)
- net VDC2_IN: now reaches F2.2, J8.1 (Pin_1)
- net VDC1_IN: now reaches F1.2, J6.1 (Pin_1)
- new net ADC_i1-: Rjp3.1, U10.8 (CH3)
- new net ADC_i2-: Rjp4.1, U10.6 (CH1)
- no-connect marks 5 -> 16
Other:
- moved on the sheet: D1, D2, D4, D5, F1, F2, J6, J7, J8, J9

Commit message: pcb first done
Parts:
- Rjp3, Rjp4: footprint Resistor_THT:R_Axial_DIN0207_L6.3mm_D2.5mm_P15.24mm_Horizontal -> Resistor_THT:R_Axial_DIN0207_L6.3mm_D2.5mm_P2.54mm_Vertical
Changed lines of the file:
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@@
 			)
 		)
-		(property "Footprint" "Resistor_THT:R_Axial_DIN0207_L6.3mm_D2.5mm_P15.24mm_Horizontal"
+		(property "Footprint" "Resistor_THT:R_Axial_DIN0207_L6.3mm_D2.5mm_P2.54mm_Vertical"
 			(at 144.78 191.008 90)
 			(hide yes)
@@
 			)
 		)
-		(property "Footprint" "Resistor_THT:R_Axial_DIN0207_L6.3mm_D2.5mm_P15.24mm_Horizontal"
+		(property "Footprint" "Resistor_THT:R_Axial_DIN0207_L6.3mm_D2.5mm_P2.54mm_Vertical"
 			(at 146.05 152.908 90)
 			(hide yes)

Commit message: modify
Connections:
- net ADC_v1: now also U4.2 (-)
- net ADC_v2: now also U4.6 (-)
- net GNDA: no longer U4.2 (-), U4.6 (-)
